File: GVS.kicad_sch (KiCad schematic)
At the start: 25 parts, among them J1 Conn_01x19_Socket, J10 Conn_01x02_Pin, J11 Conn_01x02_Pin, J2 Conn_01x02_Pin, J3 Conn_01x19_Socket, J4 Conn_01x02_Pin, J5 Conn_01x02_Pin, J6 Conn_01x19_Pin, J7 Conn_01x19_Pin, J8 Conn_01x02_Pin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

Commit message: added screw terminals
Parts:
- removed J10, J8, J9: Conn_01x02_Pin, Connector_PinHeader_2.54mm:PinHeader_1x02_P2.54mm_Vertical, symbol Connector:Conn_01x02_Pin
- added J12, J8, J9: Screw_Terminal_01x02, TerminalBlock:TerminalBlock_Xinya_XY308-2.54-2P_1x02_P2.54mm_Horizontal, symbol Connector:Screw_Terminal_01x02
Connections:
- net +12V: now also J12.1 (Pin_1)
- net 3mA limit: now also J9.1 (Pin_1)
- net A_OUT: now also J8.1 (Pin_1)
- net B_OUT: now also J8.2 (Pin_2)
- net GND: now also J12.2 (Pin_2), J9.2 (Pin_2)
